File: Mountingboard/AirOwl_v1/AirOwl_v1.kicad_pcb (KiCad board)
At the start: 2 copper layers, 49.6 x 109.8 mm, 15 parts, among them J1 USB_C_Receptacle_PowerOnly_6P, J2 Conn_01x06, J3 Conn_01x02, J4 USB_C_Receptacle_PowerOnly_6P, U1 CoreSE

Commit message: PCB renders
Parts:
- removed J1: USB_C_Receptacle_PowerOnly_6P, USB_Connectors:USB-C_6P_Vertical_THT
- added R3: 10K, Resistor_SMD:R_0805_2012Metric_Pad1.20x1.40mm_HandSolder, B.Cu at (81.3, 98.7)
- added R4: 10K, Resistor_SMD:R_0805_2012Metric_Pad1.20x1.40mm_HandSolder, B.Cu at (94.9, 98.7)
Connections:
- J4 pad A5: unconnected-(J4-CC1-PadA5) -> Net-(J4-CC1)
- J4 pad B5: unconnected-(J4-CC2-PadB5) -> Net-(J4-CC2)
Routing:
- net Net-(J4-CC1): track 0.00 -> 11.4 mm
- net Net-(J4-CC2): track 0.00 -> 11.0 mm
- net GND: vias 3 -> 9
