File: Mountingboard/AirOwl_v1/AirOwl_v1.kicad_sch (KiCad schematic)
At the start: 9 parts, among them J1 USB_C_Receptacle_PowerOnly_6P, J2 Conn_01x06, J3 Conn_01x02, J4 USB_C_Receptacle_PowerOnly_6P, U1 CoreSE

Commit message: PCB renders
Parts:
- removed J1: USB_C_Receptacle_PowerOnly_6P, USB_Connectors:USB-C_6P_Vertical_THT, symbol Connector:USB_C_Receptacle_PowerOnly_6P
- added R3, R4: 10K, Resistor_SMD:R_0805_2012Metric_Pad1.20x1.40mm_HandSolder, symbol Device:R_Small
Connections:
- net GND: now also R3.2, R4.2
- net at J4.A5 (CC1): now also R4.1
- net at J4.B5 (CC2): now also R3.1
- no-connect marks 6 -> 2
Other:
- note added: "Battery"
- note added: "Connectors"
- note added: "I2C Pullups (Optional)"
- note added: "M5Stack CoreS3"
- note added: "Note:"
- note added: "SN54"
- note added: "Type C Input"
- company: (none) -> Oizom Intruments Pvt Ltd
- title: (none) -> OIZOM AirOwl
- moved on the sheet: D2, J2, J3, J4, JP1, R1, R2, U1
